Commit message: add arm xacro

File: ros/src/robot_model/topower_v1.xacro (robot description, xacro)
@@ -5,4 +5,5 @@
   <xacro:include filename="$(find topower_v1)/src/robot_model/topower_v1_vehicle.urdf.xacro" />
   <xacro:include filename="$(find topower_v1)/src/robot_model/topower_v1_pan_tilt_cam.urdf.xacro" />
+  <xacro:include filename="$(find topower_v1)/src/robot_model/topower_v1_arm.urdf.xacro" />
   <joint name="joint_cam_to_platform" type="fixed">
       <parent link="vehicle_platform"/>
@@ -10,6 +11,10 @@
       <origin xyz="0 ${-0.5*(platform_y-pan_box_y)} ${0.5*platform_z}" rpy="0 0 0"/>
   </joint>
+  <joint name="joint_arm_to_body" type="fixed">
+      <parent link="vehicle_body"/>
+      <child link="arm_root"/>
+      <origin xyz="${-battery_box_radius} 0 0" rpy="0 0 0"/>
+  </joint>
   <!--
-  <xacro:include filename="$(find topower_v1)/src/robot_model/topower_v1_arm.urdf.xacro" />
   <xacro:include filename="$(find topower_v1)/src/robot_model/topower_v1.gazebo" />
   <joint name="joint_vehicle_to_arm" type="fixed">

File: ros/src/robot_model/topower_v1_common.xacro (robot description, xacro)
@@ -13,8 +13,13 @@
         </visual>
     </xacro:macro>
-    <xacro:macro name="box_link" params="name size_x size_y size_z mass material">
+    <xacro:macro name="box_link" params="name size_x size_y size_z mass material ori:='' ">
         <link name="${name}">
             <xacro:visualAsCollision>
-                <origin xyz="0 0 0" rpy="0 0 0"/>
+                <xacro:if value="${ori == '' }">
+                    <origin xyz="0 0 0" rpy="0 0 0"/>
+                </xacro:if>
+                <xacro:unless value="${ori == '' }">
+                    <origin xyz="${ori}" rpy="0 0 0"/>
+                </xacro:unless>
                 <geometry>
                     <box size="${size_x} ${size_y} ${size_z}"/>
