Commit message: add gazebo launch file

File: ros/robot_model/topower_v1_arm.urdf.xacro (robot description, xacro)
@@ -79,6 +79,56 @@
         <axis xyz="1 0 0"/>
         <origin xyz="${0.5*gripper_x} ${gripper_offset_y} ${gripper_base_z}" rpy="0 0 0"/>
-        <limit lower="${gripper_open_dist}" upper="0" effort="100" velocity="10" />
+        <limit lower="0" upper="${gripper_open_dist}" effort="100" velocity="10" />
         <mimic joint="joint_gripper_l" multiplier="-1" offset="0" />
     </joint>
+    <transmission name="tran_arm_base">
+        <type>transmission_interface/SimpleTransmission</type>
+        <joint name="joint_arm_base">
+        <hardwareInterface>hardware_interface/EffortJointInterface</hardwareInterface>
+        </joint>
+        <actuator name="motor_arm_base">
+        <hardwareInterface>hardware_interface/EffortJointInterface</hardwareInterface>
+        <mechanicalReduction>1</mechanicalReduction>
+        </actuator>
+    </transmission>
+    <transmission name="tran_arm_a">
+        <type>transmission_interface/SimpleTransmission</type>
+        <joint name="joint_arm_a">
+        <hardwareInterface>hardware_interface/EffortJointInterface</hardwareInterface>
+        </joint>
+        <actuator name="motor_arm_a">
+        <hardwareInterface>hardware_interface/EffortJointInterface</hardwareInterface>
+        <mechanicalReduction>1</mechanicalReduction>
+        </actuator>
+    </transmission>
+    <transmission name="tran_arm_b">
+        <type>transmission_interface/SimpleTransmission</type>
+        <joint name="joint_arm_b">
+        <hardwareInterface>hardware_interface/EffortJointInterface</hardwareInterface>
+        </joint>
+        <actuator name="motor_arm_b">
+        <hardwareInterface>hardware_interface/EffortJointInterface</hardwareInterface>
+        <mechanicalReduction>1</mechanicalReduction>
+        </actuator>
+    </transmission>
+    <transmission name="tran_gripper_base">
+        <type>transmission_interface/SimpleTransmission</type>
+        <joint name="joint_gripper_base">
+        <hardwareInterface>hardware_interface/EffortJointInterface</hardwareInterface>
+        </joint>
+        <actuator name="motor_gripper_base">
+        <hardwareInterface>hardware_interface/EffortJointInterface</hardwareInterface>
+        <mechanicalReduction>1</mechanicalReduction>
+        </actuator>
+    </transmission>
+    <transmission name="tran_gripper_l">
+        <type>transmission_interface/SimpleTransmission</type>
+        <joint name="joint_gripper_l">
+        <hardwareInterface>hardware_interface/EffortJointInterface</hardwareInterface>
+        </joint>
+        <actuator name="motor_gripper_l">
+        <hardwareInterface>hardware_interface/EffortJointInterface</hardwareInterface>
+        <mechanicalReduction>1</mechanicalReduction>
+        </actuator>
+    </transmission>
 </robot>

File: ros/robot_model/topower_v1_pan_tilt_cam.urdf.xacro (robot description, xacro)
@@ -1,7 +1,11 @@
 <?xml version="1.0"?>
 <robot name="topower_v1" xmlns:xacro="http://www.ros.org/wiki/xacro">
+    <xacro:property name="pan_base_x" value="0.055"/>
+    <xacro:property name="pan_base_y" value="0.02"/>
+    <xacro:property name="pan_base_z" value="0.02"/>
+    <xacro:property name="pan_base_mass" value="0.1"/>
     <xacro:property name="pan_box_x" value="0.055"/>
     <xacro:property name="pan_box_y" value="0.045"/>
-    <xacro:property name="pan_box_z" value="0.035"/>
+    <xacro:property name="pan_box_z" value="0.005"/>
     <xacro:property name="pan_box_mass" value="0.1"/>
     <xacro:property name="tilt_base_x" value="0.055"/>
@@ -17,14 +21,21 @@
     <xacro:property name="cam_mass" value="0.02"/>
     <!-- ==================body======================= -->
-    <link name="pan_tilt_base" />
+    <link name="pan_tilt_root" />
+    <xacro:box_link name="pan_base" size_x="${pan_base_x}" size_y="${pan_base_y}" size_z="${pan_base_z}" mass="${pan_base_mass}" material="white"/>
     <xacro:box_link name="pan_box" size_x="${pan_box_x}" size_y="${pan_box_y}" size_z="${pan_box_z}" mass="${pan_box_mass}" material="white"/>
     <xacro:box_link name="tilt_base" size_x="${tilt_base_x}" size_y="${tilt_base_y}" size_z="${tilt_base_z}" mass="${tilt_base_mass}" material="white"/>
     <xacro:box_link name="tilt_box" size_x="${tilt_box_x}" size_y="${tilt_box_y}" size_z="${tilt_box_z}" mass="${tilt_box_mass}" material="orange"/>
-    <xacro:cylinder_link name="cam" radius="${cam_radius}" height="${cam_height}" mass="${cam_mass}" material="orange"/>
+    <xacro:cylinder_link name="camera_link" radius="${cam_radius}" height="${cam_height}" mass="${cam_mass}" material="orange"/>
+    <link name="camera_link_optical" />
+    <joint name="joint_pan_tilt_root_to_pan_base" type="fixed">
+        <parent link="pan_tilt_root"/>
+        <child link="pan_base"/>
+        <origin xyz="0 0 ${0.5*pan_base_z}" rpy="0 0 0"/>
+    </joint>
     <joint name="joint_cam_pan" type="revolute">
-        <parent link="pan_tilt_base"/>
+        <parent link="pan_base"/>
         <child link="pan_box"/>
         <axis xyz="0 0 1"/>
-        <origin xyz="0 0 ${0.5*pan_box_z}" rpy="0 0 0"/>
+        <origin xyz="0 0 ${0.5*(pan_base_z+pan_box_z)}" rpy="0 0 0"/>
         <limit lower="${-2*PI/3}" upper="${2*PI/3}" effort="100" velocity="10" />
     </joint>
@@ -43,6 +54,11 @@
     <joint name="joint_tilt_base_to_cam" type="fixed">
         <parent link="tilt_box"/>
-        <child link="cam"/>
+        <child link="camera_link"/>
         <origin xyz="${0.5*(tilt_box_x+cam_height)} 0 0" rpy="0 ${0.5*PI} 0"/>
+    </joint>
+    <joint name="joint_cam_to_optical" type="fixed">
+        <parent link="camera_link"/>
+        <child link="camera_link_optical"/>
+        <origin xyz="0 0 ${0.5*cam_height}" rpy="0 ${-0.5*PI} 0"/>
     </joint>
     <!-- ======================transitions=============================-->
@@ -50,8 +66,8 @@
         <type>transmission_interface/SimpleTransmission</type>
         <joint name="joint_cam_pan">
-        <hardwareInterface>hardware_interface/PositionJointInterface</hardwareInterface>
+        <hardwareInterface>hardware_interface/EffortJointInterface</hardwareInterface>
         </joint>
         <actuator name="motor_cam_pan">
-        <hardwareInterface>hardware_interface/PositionJointInterface</hardwareInterface>
+        <hardwareInterface>hardware_interface/EffortJointInterface</hardwareInterface>
         <mechanicalReduction>1</mechanicalReduction>
         </actuator>
@@ -60,8 +76,8 @@
         <type>transmission_interface/SimpleTransmission</type>
         <joint name="joint_cam_tilt">
-        <hardwareInterface>hardware_interface/PositionJointInterface</hardwareInterface>
+        <hardwareInterface>hardware_interface/EffortJointInterface</hardwareInterface>
         </joint>
         <actuator name="motor_cam_tilt">
-        <hardwareInterface>hardware_interface/PositionJointInterface</hardwareInterface>
+        <hardwareInterface>hardware_interface/EffortJointInterface</hardwareInterface>
         <mechanicalReduction>1</mechanicalReduction>
         </actuator>

Commit message: adjust pid parameter

File: ros/robot_model/topower_v1_arm.urdf.xacro (robot description, xacro)
@@ -44,5 +44,5 @@
         <axis xyz="0 0 1"/>
         <origin xyz="0 0 ${0.5*(battery_box_height+arm_base_height)}" rpy="0 0 0"/>
-        <limit lower="${-PI}" upper="${PI}" effort="100" velocity="10" />
+        <limit lower="${-PI}" upper="${PI}" effort="12" velocity="0.9" />
     </joint>
     <joint name="joint_arm_a" type="revolute">
@@ -51,5 +51,5 @@
         <axis xyz="1 0 0"/>
         <origin xyz="0 0 ${0.5*arm_base_height}" rpy="0 0 0"/>
-        <limit lower="${-0.5*PI}" upper="${0.5*PI}" effort="100" velocity="10" />
+        <limit lower="${-0.5*PI}" upper="${0.5*PI}" effort="12" velocity="0.9" />
     </joint>
     <joint name="joint_arm_b" type="revolute">
@@ -58,5 +58,5 @@
         <axis xyz="1 0 0"/>
         <origin xyz="0 0 ${arm_a_z}" rpy="0 0 0"/>
-        <limit lower="${-0.5*PI}" upper="${0.5*PI}" effort="100" velocity="10" />
+        <limit lower="${-0.5*PI}" upper="${0.5*PI}" effort="10" velocity="0.9" />
     </joint>
     <joint name="joint_gripper_base" type="revolute">
@@ -65,5 +65,5 @@
         <axis xyz="1 0 0"/>
         <origin xyz="0 ${gripper_base_offset_y} ${arm_b_z}" rpy="0 0 0"/>
-        <limit lower="${-0.5*PI}" upper="${0.5*PI}" effort="100" velocity="10" />
+        <limit lower="${-0.5*PI}" upper="${0.5*PI}" effort="12" velocity="0.9" />
     </joint>
     <joint name="joint_gripper_l" type="prismatic">
@@ -72,5 +72,5 @@
         <axis xyz="1 0 0"/>
         <origin xyz="${-0.5*gripper_x} ${gripper_offset_y} ${gripper_base_z}" rpy="0 0 0"/>
-        <limit lower="${-gripper_open_dist}" upper="0" effort="100" velocity="10" />
+        <limit lower="${-gripper_open_dist}" upper="0" effort="12" velocity="0.9" />
     </joint>
     <joint name="joint_gripper_r" type="prismatic">
@@ -79,5 +79,5 @@
         <axis xyz="1 0 0"/>
         <origin xyz="${0.5*gripper_x} ${gripper_offset_y} ${gripper_base_z}" rpy="0 0 0"/>
-        <limit lower="0" upper="${gripper_open_dist}" effort="100" velocity="10" />
+        <limit lower="0" upper="${gripper_open_dist}" effort="12" velocity="0.9" />
         <mimic joint="joint_gripper_l" multiplier="-1" offset="0" />
     </joint>
