Commit message: add moveit control to arm hardware

File: topower_v1/robot_model/topower_v1_arm.urdf.xacro (robot description, xacro)
@@ -44,5 +44,5 @@
         <axis xyz="0 0 1"/>
         <origin xyz="0 0 ${0.5*(battery_box_height+arm_base_height)}" rpy="0 0 0"/>
-        <limit lower="${-PI}" upper="${PI}" effort="12" velocity="0.9" />
+        <limit lower="${-0.5*PI}" upper="${0.5*PI}" effort="12" velocity="0.9" />
     </joint>
     <joint name="joint_arm_a" type="revolute">
