Commit message: control arm directly from action client for faster response when moving using joystick

File: topower_v1/robot_model/topower_v1_pan_tilt_cam.urdf.xacro (robot description, xacro)
@@ -17,6 +17,5 @@
     <xacro:property name="tilt_box_z" value="0.03"/>
     <xacro:property name="tilt_box_mass" value="0.05"/>
-    <xacro:property name="cam_radius" value="0.01"/>
-    <xacro:property name="cam_height" value="0.01"/>
+    <xacro:property name="cam_box_size" value="0.01"/>
     <xacro:property name="cam_mass" value="0.02"/>
     <!-- ==================body======================= -->
@@ -26,5 +25,5 @@
     <xacro:box_link name="tilt_base" size_x="${tilt_base_x}" size_y="${tilt_base_y}" size_z="${tilt_base_z}" mass="${tilt_base_mass}" material="white"/>
     <xacro:box_link name="tilt_box" size_x="${tilt_box_x}" size_y="${tilt_box_y}" size_z="${tilt_box_z}" mass="${tilt_box_mass}" material="orange"/>
-    <xacro:cylinder_link name="camera_link" radius="${cam_radius}" height="${cam_height}" mass="${cam_mass}" material="orange"/>
+    <xacro:box_link name="camera_link" size_x="${cam_box_size}" size_y="${cam_box_size}" size_z="${cam_box_size}" mass="${cam_mass}" material="orange"/>
     <link name="camera_link_optical" />
     <joint name="joint_pan_tilt_root_to_pan_base" type="fixed">
@@ -55,10 +54,10 @@
         <parent link="tilt_box"/>
         <child link="camera_link"/>
-        <origin xyz="${0.5*(tilt_box_x+cam_height)} 0 0" rpy="0 ${0.5*PI} 0"/>
+        <origin xyz="${0.5*(tilt_box_x+cam_box_size)} 0 0" rpy="0 0 0"/>
     </joint>
     <joint name="joint_cam_to_optical" type="fixed">
         <parent link="camera_link"/>
         <child link="camera_link_optical"/>
-        <origin xyz="0 0 ${0.5*cam_height}" rpy="0 ${-0.5*PI} 0"/>
+        <origin xyz="0 0 ${0.5*cam_box_size}" rpy="0 0 0"/>
     </joint>
     <!-- ======================transitions=============================-->
